Commit message: Three sensors working

File: hdf_model/robots/hdf_model.urdf (robot description, URDF)
Before this commit: robot hdf_model, 7 links, 6 joints
Links:
- added link ultrasonic_link_centre, mass 1.0; collision box size=0.045 0.02 0.001; visual box size=0.001 0.045 0.02
- added link ultrasonic_link_left_1, mass 1.0; collision box size=0.045 0.02 0.001; visual box size=0.001 0.045 0.02
Joints:
- added joint ultrasonic_joint_centre_1: type fixed, parent base_link, child ultrasonic_link_centre, origin xyz=-0.26 0 0.005 rpy=0 0 3.22886, axis 0 0 0
- added joint ultrasonic_joint_left_1: type fixed, parent base_link, child ultrasonic_link_left_1, origin xyz=-0.13 -0.26 0.005 rpy=0 0 4.88692, axis 0 0 0

Commit message: Third one-Right side rought added sensors, left side shud define the joint values tmrw

File: hdf_model/robots/hdf_model.urdf (robot description, URDF)
Before this commit: robot hdf_model, 9 links, 8 joints
Links:
- added link ultrasonic_link_left_2, mass 0.1; collision box size=0.045 0.02 0.001; visual box size=0.001 0.045 0.02
- added link ultrasonic_link_left_3, mass 0.1; collision box size=0.045 0.02 0.001; visual box size=0.001 0.045 0.02
- added link ultrasonic_link_right_2, mass 0.1; collision box size=0.045 0.02 0.001; visual box size=0.001 0.045 0.02
- added link ultrasonic_link_right_3, mass 0.1; collision box size=0.045 0.02 0.001; visual box size=0.001 0.045 0.02
- link ultrasonic_link_left_1: mass 1.0 -> 0.1
- link ultrasonic_link_right_1: mass 1.0 -> 0.1
Joints:
- added joint ultrasonic_joint_left_2: type fixed, parent base_link, child ultrasonic_link_left_2, origin xyz=-0.13 -0.26 0.005 rpy=0 0 4.88692, axis 0 0 0
- added joint ultrasonic_joint_left_3: type fixed, parent base_link, child ultrasonic_link_left_3, origin xyz=-0.13 -0.26 0.005 rpy=0 0 4.88692, axis 0 0 0
- added joint ultrasonic_joint_right_2: type fixed, parent base_link, child ultrasonic_link_right_2, origin xyz=-0.13 0.26 0.005 rpy=0 0 2.0944, axis 0 0 0
- added joint ultrasonic_joint_right_3: type fixed, parent base_link, child ultrasonic_link_right_3, origin xyz=0.08 0.23 0.005 rpy=0 0 -2.0944, axis 0 0 0
- joint ultrasonic_joint_right_1: origin xyz=-0.13 0.26 0.005 rpy=0 0 2.0944 -> xyz=-0.22 0.13 0.005 rpy=0 0 2.61799
